File: hardware/kicad/beamformer/beamformer.kicad_sch (KiCad schematic)
At the start: 19 parts, among them J1 SWD_HEADER, J2 USB_C_Receptacle_USB2.0_16P, U1 STM32H753ZITx, U2 USBLC6-2SC6, U3 TLC59116FIPWR, U4 ADAU7118ACPZRL, U5 MCP1826S-3302E/DB, U6 TLV75518PDBVR, U7 SN74AXC4T774PWR, Y1 16 MHz

Commit message: schematic progress
Parts:
- added C1, C10, C11, C12, C13, C14, C15, C16, C17, C18, C19, C2, C22, C23, C8, C9: 0.1uF, Capacitor_SMD:C_0805_2012Metric, symbol Device:C
- added C20, C21: 10pF, Capacitor_SMD:C_0805_2012Metric, symbol Device:C
- added C3: 10uF, Capacitor_SMD:C_0805_2012Metric, symbol Device:C
- added C4, C5, C6, C7: 1uF, Capacitor_SMD:C_0805_2012Metric, symbol Device:C
- added D10, D11, D12, D13, D14, D15, D16, D2, D3, D4, D5, D6, D7, D8, D9: LED_Blue_AA4040QBS-G, Beamformer:LED_Kingbright_AA4040QBS-G, symbol Device:LED
- added R1, R10, R11, R12, R13, R14, R15, R16, R2, R3, R4, R5, R6, R7, R8, R9: 220R, Resistor_SMD:R_0805_2012Metric, symbol Device:R
- added R17, R20: 4K7, Resistor_SMD:R_0805_2012Metric, symbol Device:R
- added R18: 10K, Resistor_SMD:R_0805_2012Metric, symbol Device:R
- added R19: 2K2, Resistor_SMD:R_0805_2012Metric, symbol Device:R
- added R21, R22: 5K1, Resistor_SMD:R_0805_2012Metric, symbol Device:R
- D1: value LED -> LED_Blue_AA4040QBS-G; footprint PW0016A_N -> Beamformer:LED_Kingbright_AA4040QBS-G
Connections:
- net GND: now also J1.2 (Pin_2), J2.A1 (GND), J2.A12 (GND), J2.B1 (GND), J2.B12 (GND), J2.SH (SHIELD), MK1.2 (SELECT), MK1.5 (THSEL), MK2.5 (THSEL), MK3.2 (SELECT), MK3.5 (THSEL), MK4.5 (THSEL), MK5.2 (SELECT), MK5.5 (THSEL), MK6.5 (THSEL), MK7.2 (SELECT), MK7.5 (THSEL), MK8.5 (THSEL), U2.2 (GND), U3.10 (GND), U3.19 (GND), U3.2 (A0), U3.24 (GND), U3.3 (A1), U3.4 (A2), U3.5 (A3), U4.15 (GND), U4.17 (EPAD), U4.8 (SDA), U5.2 (GND), U6.2 (GND), U7.10 (GND), U7.2 (DIR2), U7.7 (DIR3), U7.8 (DIR4), U7.9 (OE_N), C1.1, C10.2, C11.2, C12.2, C13.2, C14.2, C15.2, C16.2, C17.2, C18.1, C19.1, C2.1, C20.1, C21.1, C22.2, C23.2, C3.2, C4.2, C5.2, C6.1, C7.1, C8.2, C9.2, R19.1, R21.2, R22.1
- net +3V3: now reaches U3.28 (VCC)
- net +3V3: now also J1.1 (Pin_1), U1.6 (VBAT), U5.3 (VO), U6.1 (IN), U6.3 (EN), U7.15 (VCCB), C19.2, C5.1, C6.2, R17.2, R18.1, R20.1
- net +5V: now reaches J2.A4 (VBUS), J2.A9 (VBUS), J2.B4 (VBUS), J2.B9 (VBUS)
- net +5V: now also U2.5 (VBUS), U5.1 (VI), C4.1, R1.2, R10.2, R11.2, R12.2, R13.2, R14.2, R15.2, R16.2, R2.2, R3.2, R4.2, R5.2, R6.2, R7.2, R8.2, R9.2
- net at J2.A5 (CC1): now also R21.1
- net at J2.A6 (D+): now also J2.B6 (D+), U2.1 (I/O1)
- net at J2.A7 (D-): now also J2.B7 (D-), U2.3 (I/O2)
- net at J2.B5 (CC2): now also R22.2
- net +1V8: now reaches U7.1 (DIR1)
- net +1V8: now also MK1.7 (VDD), MK2.2 (SELECT), MK2.7 (VDD), MK3.7 (VDD), MK4.2 (SELECT), MK4.7 (VDD), MK5.7 (VDD), MK6.2 (SELECT), MK6.7 (VDD), MK7.7 (VDD), MK8.2 (SELECT), MK8.7 (VDD), U4.13 (EN), U4.14 (DVDD), U4.16 (IOVDD), U4.7 (SCL), U6.5 (OUT), U7.16 (VCCA), C10.1, C11.1, C12.1, C13.1, C14.1, C15.1, C16.1, C17.1, C18.2, C7.2, C8.1, C9.1
- net at U7.12 (B3): now also U1.3 (PE4)
- net at U7.13 (B2): now also U1.4 (PE5)
- net at U7.14 (B1): now also U1.5 (PE6)
- net at U7.3 (A1): now also U4.11 (SDATA)
- net at U7.4 (A2): now also U4.10 (BCLK)
- net at U7.5 (A3): now also U4.9 (FSYNC)
- net at MK5.1 (DATA): now also MK6.1 (DATA), U4.5 (PDM_DAT2)
- net at MK5.6 (CLK): now also MK6.6 (CLK), MK7.6 (CLK), MK8.6 (CLK), U4.4 (PDM_CLK1)
- net at MK2.1 (DATA): now also MK1.1 (DATA), U4.2 (PDM_DAT0)
- net at MK2.6 (CLK): now also MK1.6 (CLK), MK3.6 (CLK), MK4.6 (CLK), U4.1 (PDM_CLK0)
- net at D1.1 (K): now also U3.6 (*OUT0)
- net at D1.2 (A): now also R1.1
- net at U4.3 (PDM_DAT1): now also MK3.1 (DATA), MK4.1 (DATA)
- net at U4.6 (PDM_DAT3): now also MK7.1 (DATA), MK8.1 (DATA)
- net at U1.103 (PA11): now also U2.4 (I/O2)
- net at U1.104 (PA12): now also U2.6 (I/O1)
- net at U1.105 (PA13): now also J1.3 (Pin_3)
- net at U1.109 (PA14): now also J1.4 (Pin_4)
- net at U1.136 (PB6): now also U3.26 (SCL), R17.1
- net at U1.137 (PB7): now also U3.27 (SDA), R20.2
- net at U1.25 (NRST): now also J1.5 (Pin_5), C2.2
- net at U1.71 (VCAP): now also C22.1
- net at Y1.1: now also C21.2
- net at Y1.2: now also C20.2
- net at U3.1 (REXT): now also R19.2
- net at U3.11 (*OUT4): now also D5.1 (K)
- net at U3.12 (*OUT5): now also D6.1 (K)
- net at U3.13 (*OUT6): now also D7.1 (K)
- net at U3.14 (*OUT7): now also D8.1 (K)
- net at U3.15 (*OUT8): now also D9.1 (K)
- net at U3.16 (*OUT9): now also D10.1 (K)
- net at U3.17 (*OUT10): now also D11.1 (K)
- net at U3.18 (*OUT11): now also D12.1 (K)
- net at U3.25 (*RESET): now also R18.2
- net at U3.7 (*OUT1): now also D2.1 (K)
- net at U3.8 (*OUT2): now also D3.1 (K)
- net at U3.9 (*OUT3): now also D4.1 (K)
- new net: D11.2 (A), R11.1
- new net: D14.2 (A), R14.1
- new net: D7.2 (A), R7.1
- new net: D2.2 (A), R2.1
- new net: D5.2 (A), R5.1
- new net: D4.2 (A), R4.1
- new net: D8.2 (A), R8.1
- new net: D9.2 (A), R9.1
- new net: D16.2 (A), R16.1
- new net: D15.2 (A), R15.1
- new net: D10.2 (A), R10.1
- new net: D6.2 (A), R6.1
- new net: D12.2 (A), R12.1
- new net: D3.2 (A), R3.1
- new net: D13.2 (A), R13.1
- no-connect marks 0 -> 10
Other:
- moved on the sheet: D1, J1, J2, MK1, MK2, MK3, MK4, MK5, MK6, MK7, MK8, U1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

Commit message: final schematic version and pcb update
Parts:
- removed R19: 2K2, Resistor_SMD:R_0805_2012Metric, symbol Device:R
- added C24, C25, C26, C27, C28, C29, C30, C31, C32, C33, C34, C35, C37, C39: 0.1uF, Capacitor_SMD:C_0805_2012Metric, symbol Device:C
- added C36, C38: 1uF, Capacitor_SMD:C_0805_2012Metric, symbol Device:C
- added C40: 4.7uF, Capacitor_SMD:C_0805_2012Metric, symbol Device:C
- added R23: 10K, Resistor_SMD:R_0805_2012Metric, symbol Device:R
- C22, C23: value 0.1uF -> 2.2uF
- C3: value 10uF -> 4.7uF
- U4: footprint Package_CSP:LFCSP-16-1EP_3x3mm_P0.5mm_EP1.6x1.6mm -> Beamformer:CP-16-22_ADI
Connections:
- net +3V3: now also C1.2, U1.108 (VDD), U1.121 (VDD), U1.131 (VDD), U1.143 (PDR_ON), U1.144 (VDD), U1.17 (VDD), U1.30 (VDD), U1.32 (VREF+), U1.33 (VDDA), U1.39 (VDD), U1.52 (VDD), U1.62 (VDD), U1.72 (VDD), U1.84 (VDD), U1.95 (VDD33_USB), C24.2, C25.2, C26.2, C27.2, C28.2, C29.2, C30.1, C31.2, C32.2, C33.2, C34.2, C35.2, C36.2, C37.2, C38.1, C39.1, C40.2
- net +5V: now also C3.1
- net GND: now also U1.107 (VSS), U1.120 (VSS), U1.130 (VSS), U1.16 (VSS), U1.31 (VSSA), U1.38 (VSS), U1.51 (VSS), U1.61 (VSS), U1.83 (VSS), U1.94 (VSS), C24.1, C25.1, C26.1, C27.1, C28.1, C29.1, C30.2, C31.1, C32.1, C33.1, C34.1, C35.1, C36.1, C37.1, C38.2, C39.2, C40.1, R23.1
- net NRST: now also C2.2, J1.5 (Pin_5), U1.25 (NRST)
- net SWCLK: now also J1.4 (Pin_4), U1.109 (PA14)
- net SWDIO: now also J1.3 (Pin_3), U1.105 (PA13)
- net at D11.1 (K): now also U3.20 (*OUT12); no longer U3.17 (*OUT10)
- net at D14.1 (K): now also U3.18 (*OUT11)
- net at C22.1, U1.71 (VCAP): now also C23.1, U1.106 (VCAP)
- net at U3.13 (*OUT6): now also D6.1 (K); no longer D7.1 (K)
- net at D16.1 (K): now also U3.23 (*OUT15)
- net at C21.2, Y1.1: now also U1.24 (PH1)
- net at D15.1 (K): now also U3.21 (*OUT13)
- net at U1.138 (BOOT0): now also R23.2
- net at U1.23 (PH0): now also C20.2, Y1.2
- net at U3.12 (*OUT5): now also D7.1 (K); no longer D6.1 (K)
- net at U3.16 (*OUT9): now also D13.1 (K); no longer D10.1 (K)
- net at D12.1 (K): now also U3.22 (*OUT14); no longer U3.18 (*OUT11)
- new net: D10.1 (K), U3.17 (*OUT10)
- no-connect marks 10 -> 117
Other:
- moved on the sheet: C1, C2, C3, D1, D2, J1, J2, R1, R17, R2, R20, R21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

Commit message: pcb wiring started
Parts:
- J2: footprint Connector_USB:USB_C_Receptacle_GCT_USB4085 -> Beamformer:USB_C_Receptacle_GCT_USB4085
Changed lines of the file:
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@@
 			)
 		)
-		(property "Footprint" "Connector_USB:USB_C_Receptacle_GCT_USB4085"
+		(property "Footprint" "Beamformer:USB_C_Receptacle_GCT_USB4085"
 			(at 334.01 86.36 0)
 			(hide yes)

Commit message: PCB complete
Parts:
- removed J2: USB_C_Receptacle_USB2.0_16P, Beamformer:USB_C_Receptacle_GCT_USB4085, symbol Connector:USB_C_Receptacle_USB2.0_16P
- added J2: USB4145-03-0170-C, Beamformer:CONN_USB4145-03-0230-C_GCT, symbol USB4145-03-0170-C:USB4145-03-0170-C
- added J3: Audio/UART Header, Connector_PinHeader_2.54mm:PinHeader_1x06_P2.54mm_Vertical, symbol Connector_Generic:Conn_01x06
- added TP1, TP10, TP11, TP12, TP13, TP2, TP3, TP4, TP5, TP6, TP7, TP8, TP9: TestPoint, TestPoint:TestPoint_Pad_D1.5mm, symbol Connector:TestPoint
Connections:
- net +1V8: now also TP10.1
- net +3V3: now also TP11.1
- net +5V: now also C3.2, J2.A4 (VBUS_1), J2.A9 (VBUS_2), J2.B4 (VBUS_3), J2.B9 (VBUS_4), TP12.1; no longer C3.1
- net GND: now also C3.1, R22.2, J2.1 (MH1), J2.2 (MH2), J2.3 (MH3), J2.4 (MH4), J2.A1 (GND_1), J2.A12 (GND_2), J2.B1 (GND_3), J2.B12 (GND_4), J3.1 (Pin_1), TP1.1, TP13.1, TP5.1, TP9.1; no longer C3.2, R22.1
- net at R21.1: now also J2.B5 (CC2)
- net at U2.1 (I/O1): now also J2.A6 (DP1), J2.B6 (DP2)
- net at U2.3 (I/O2): now also J2.A7 (DN1), J2.B7 (DN2)
- net SDATA: now reaches U4.11 (SDATA), U7.3 (A1)
- net SDATA: now also J3.4 (Pin_4)
- net BCLCK: now reaches U4.10 (BCLK), U7.4 (A2)
- net BCLCK: now also J3.3 (Pin_3)
- net FSYNC: now reaches U4.9 (FSYNC), U7.5 (A3)
- net FSYNC: now also J3.2 (Pin_2)
- net at MK5.1 (DATA), MK6.1 (DATA), U4.5 (PDM_DAT2): now also TP6.1
- net at MK5.6 (CLK), MK6.6 (CLK), MK7.6 (CLK)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: now also TP8.1
- net at MK1.1 (DATA), MK2.1 (DATA), U4.2 (PDM_DAT0): now also TP2.1
- net at MK1.6 (CLK), MK2.6 (CLK), MK3.6 (CLK)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: now also TP4.1
- net at MK3.1 (DATA), MK4.1 (DATA), U4.3 (PDM_DAT1): now also TP3.1
- net at MK7.1 (DATA), MK8.1 (DATA), U4.6 (PDM_DAT3): now also TP7.1
- net TX: now reaches U1.69 (PB10)
- net TX: now also J3.6 (Pin_6)
- net RX: now reaches U1.70 (PB11)
- net RX: now also J3.5 (Pin_5)
- new net: J2.A5 (CC1), R22.1
- no-connect marks 117 -> 115
Other:
- moved on the sheet: C3, R21, R22
